File: Hardware/Qwiic_Differential_Pressure_Sensor-SDP31.brd (EAGLE design)
At the start: 25.4 x 25.4 mm, 51 parts, among them J2 QWIIC_RIGHT_ANGLE, J4 QWIIC_RIGHT_ANGLE, U1 SDP31

Commit message: Change IRQ to INT. Add Address label.
Parts:
- added U$21: (no value), output:#ADDRESS#0
- U$5, U$6: device output:#IRQ#0 -> output:##INT##0
- moved U$14 2.69 mm to (6.35, 15.9), turned to 0 degrees
- moved C1 0.25 mm to (12.7, 14.9)
Connections:
- net IRQ renamed !INT!
