File: Hardware/Qwiic_Differential_Pressure_Sensor-SDP31.brd (EAGLE design)
At the start: 25.4 x 25.4 mm, 52 parts, among them J2 QWIIC_RIGHT_ANGLE, J4 QWIIC_RIGHT_ANGLE, U1 SDP31

Commit message: Update PROD_IDs. Delete New-Parts
Parts:
- JP1, JP2, JP5, JP6: device SparkFun:MICRO-FIDUCIAL -> SparkFun-Aesthetics:FIDUCIAL-MICRO
- JP3, JP4: device SparkFun:STAND-OFF -> SparkFun-Hardware:STAND-OFF
- R4: value 1.2K -> 1.20k; device New-Parts_SparkFun-Resistors:0603 -> SparkFun-Resistors:0603
- R5: value 2.7K -> 2.7k; device New-Parts_SparkFun-Resistors:0603 -> SparkFun-Resistors:0603
- U1: device New-Parts_SparkFun-Sensors:SDP31 -> SparkFun-Sensors:SDP3X
